File: Arduino.kicad_pcb (KiCad board)
At the start: 2 copper layers, 17 parts, among them J1 Serial, J2 Digital pins, J3 ICSP connector, J4 I2C, U1 DS1337_AH, U2 24LC1025, U3 24LC1025, U4 ATMEGA328P-AU, Y1 Crystal 32MHZ, Y2 Crystal 16MHZ

Commit message: Complete the placement
Parts:
- moved BT1 97.1 mm to (147.8, 68.0)
- moved R2 96.9 mm to (153.0, 67.7), turned to 180 degrees
- moved Y2 91.1 mm to (155.7, 71.6)
- moved C2 85.4 mm to (163.7, 69.2)
- moved C1 75.4 mm to (163.7, 72.4)
- moved D1 68.9 mm to (180.0, 85.8)
- moved U4 66.6 mm to (159.0, 80.4)
- moved U2 65.2 mm to (171.7, 74.7)
- moved C3 62.8 mm to (180.0, 81.3), turned to 180 degrees
- moved R1 62.3 mm to (184.9, 85.8), turned to 180 degrees
- moved U1 54.5 mm to (182.1, 72.6)
- moved U3 53.5 mm to (171.7, 82.1)
- moved Y1 48.3 mm to (184.8, 81.3)
- moved J3 41.7 mm to (150.3, 79.1)
- moved J2 40.9 mm to (155.0, 89.4), turned to 90 degrees
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